File: generic-pcb.kicad_pcb (KiCad board)
At the start: 2 copper layers, 99.1 x 99.1 mm, 239 parts

Commit message: Create version with disconnected rails
Parts:
- removed the REF**8 at (181.6, 61.0)
- removed the REF**8 at (135.9, 61.0)
- added REF**8: GND bus, generic-pcb:gnd-bus, F.Cu at (181.6, 61.0)
- added REF**8: GND bus, generic-pcb:gnd-bus, F.Cu at (135.9, 61.0)
Other:
- board text added: "Protoboard (C) 2015 Rich Wareham, CC BY-SA. Modifications by Alexis Lockwood, 2020."
- board text added: "https://github.com/alexisvl/protoboard-pcb / https://github.com/rjw57/protoboard-pcb"
- board text removed: "Gnd"
- board text removed: "Protoboard (C) 2015 Rich Wareham, CC BY-SA"
- board text removed: "https://github.com/rjw57/protoboard-pcb"
